File: hard/insect-robot.sch (EAGLE design)
At the start: 13 parts, among them Q1 AO3400, SW1 SWITCH-DT, U1 ATMEGA328P-QFN32, U2 PW0316

Commit message: Route some wires
Parts:
- BAT1: value BATTERY-SMD -> BATTERY-SMD-SMALL; device MyLibrary:BATTERY-SMD -> MyLibrary:BATTERY-SMD-SMALL
Connections:
- net B-: now also RP1A.1; no longer RP1C.1
- net R-: now also RP1C.1; no longer RP1A.1
- net RB-: now also RP1A.2; no longer RP1C.2
- net RR-: now also RP1C.2; no longer RP1A.2
Other:
- moved on the sheet: RP1A, RP1C
Changed lines of the file:
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@@
 <part name="SUPPLY1" library="MyLibrary" deviceset="VBAT" device=""/>
 <part name="SUPPLY2" library="MyLibrary" deviceset="GND" device=""/>
-<part name="BAT1" library="MyLibrary" deviceset="BATTERY" device="-SMD"/>
+<part name="BAT1" library="MyLibrary" deviceset="BATTERY" device="-SMD-SMALL" value="BATTERY-SMD-SMALL"/>
 <part name="SUPPLY3" library="MyLibrary" deviceset="VBAT" device=""/>
 <part name="SUPPLY4" library="MyLibrary" deviceset="GND" device=""/>
@@
 <instance part="C1" gate="A" x="-35.56" y="2.54" rot="R90"/>
 <instance part="SUPPLY10" gate="GND" x="-43.18" y="2.54" rot="R270"/>
-<instance part="RP1" gate="A" x="40.64" y="-5.08" smashed="yes">
-<attribute name="NAME" x="43.18" y="-5.08" size="1.778" layer="95"/>
-<attribute name="VALUE" x="50.8" y="-5.08" size="1.778" layer="96"/>
+<instance part="RP1" gate="A" x="40.64" y="-10.16" smashed="yes">
+<attribute name="NAME" x="43.18" y="-10.16" size="1.778" layer="95"/>
+<attribute name="VALUE" x="50.8" y="-10.16" size="1.778" layer="96"/>
 </instance>
 <instance part="RP1" gate="B" x="40.64" y="-7.62" smashed="yes">
@@
 <attribute name="VALUE" x="50.8" y="-7.62" size="1.778" layer="96"/>
 </instance>
-<instance part="RP1" gate="C" x="40.64" y="-10.16" smashed="yes">
-<attribute name="NAME" x="43.18" y="-10.16" size="1.778" layer="95"/>
-<attribute name="VALUE" x="50.8" y="-10.16" size="1.778" layer="96"/>
+<instance part="RP1" gate="C" x="40.64" y="-5.08" smashed="yes">
+<attribute name="NAME" x="43.18" y="-5.08" size="1.778" layer="95"/>
+<attribute name="VALUE" x="50.8" y="-5.08" size="1.778" layer="96"/>
 </instance>
 <instance part="RP1" gate="D" x="63.5" y="-22.86"/>
@@
 </segment>
 </net>
-<net name="R-" class="0">
-<segment>
-<pinref part="D1" gate="A" pin="R-"/>
-<wire x1="55.88" y1="-5.08" x2="45.72" y2="-5.08" width="0.1524" layer="91"/>
-<pinref part="RP1" gate="A" pin="1"/>
-</segment>
-</net>
-<net name="G-" class="0">
-<segment>
-<pinref part="D1" gate="A" pin="G-"/>
-<wire x1="55.88" y1="-7.62" x2="45.72" y2="-7.62" width="0.1524" layer="91"/>
-<pinref part="RP1" gate="B" pin="1"/>
-</segment>
-</net>
-<net name="B-" class="0">
-<segment>
-<pinref part="D1" gate="A" pin="B-"/>
-<wire x1="55.88" y1="-10.16" x2="45.72" y2="-10.16" width="0.1524" layer="91"/>
-<pinref part="RP1" gate="C" pin="1"/>
-</segment>
-</net>
 <net name="AREF" class="0">
 <segment>
 <pinref part="U1" gate="P" pin="AREF"/>
 <pinref part="C1" gate="A" pin="2"/>
-</segment>
-</net>
-<net name="RR-" class="0">
-<segment>
-<pinref part="U1" gate="P" pin="PB0(ICP1)"/>
-<pinref part="RP1" gate="A" pin="2"/>
-</segment>
-</net>
-<net name="RG-" class="0">
-<segment>
-<pinref part="U1" gate="P" pin="PB1(OC1A)"/>
-<pinref part="RP1" gate="B" pin="2"/>
-</segment>
-</net>
-<net name="RB-" class="0">
-<segment>
-<pinref part="U1" gate="P" pin="PB2(SS/OC1B)"/>
-<pinref part="RP1" gate="C" pin="2"/>
 </segment>
 </net>
@@
 </segment>
 </net>
+<net name="RR-" class="0">
+<segment>
+<pinref part="RP1" gate="C" pin="2"/>
+<pinref part="U1" gate="P" pin="PB0(ICP1)"/>
+</segment>
+</net>
+<net name="RG-" class="0">
+<segment>
+<pinref part="RP1" gate="B" pin="2"/>
+<pinref part="U1" gate="P" pin="PB1(OC1A)"/>
+</segment>
+</net>
+<net name="RB-" class="0">
+<segment>
+<pinref part="RP1" gate="A" pin="2"/>
+<pinref part="U1" gate="P" pin="PB2(SS/OC1B)"/>
+</segment>
+</net>
+<net name="R-" class="0">
+<segment>
+<pinref part="RP1" gate="C" pin="1"/>
+<pinref part="D1" gate="A" pin="R-"/>
+<wire x1="45.72" y1="-5.08" x2="55.88" y2="-5.08" width="0.1524" layer="91"/>
+</segment>
+</net>
+<net name="G-" class="0">
+<segment>
+<pinref part="RP1" gate="B" pin="1"/>
+<pinref part="D1" gate="A" pin="G-"/>
+<wire x1="45.72" y1="-7.62" x2="55.88" y2="-7.62" width="0.1524" layer="91"/>
+</segment>
+</net>
+<net name="B-" class="0">
+<segment>
+<pinref part="RP1" gate="A" pin="1"/>
+<pinref part="D1" gate="A" pin="B-"/>
+<wire x1="45.72" y1="-10.16" x2="55.88" y2="-10.16" width="0.1524" layer="91"/>
+</segment>
+</net>

Commit message: Done routing
Connections:
- removed net RST: HD2.5, U1.PC6(RESET)
- net B-: now also RP1B.1; no longer RP1A.1
- net G-: now also RP1C.1; no longer RP1B.1
- net R-: now also RP1D.1; no longer RP1C.1
- net RB-: now also RP1B.2; no longer RP1A.2
- net RG-: now also RP1C.2; no longer RP1B.2
- net RR-: now also RP1D.2; no longer RP1C.2
Other:
- moved on the sheet: RP1A, RP1B, RP1C, RP1D
Changed lines of the file:
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@@
 <instance part="C1" gate="A" x="-35.56" y="2.54" rot="R90"/>
 <instance part="SUPPLY10" gate="GND" x="-43.18" y="2.54" rot="R270"/>
-<instance part="RP1" gate="A" x="40.64" y="-10.16" smashed="yes">
+<instance part="RP1" gate="A" x="60.96" y="-22.86" smashed="yes">
+<attribute name="NAME" x="63.5" y="-22.86" size="1.778" layer="95"/>
+<attribute name="VALUE" x="71.12" y="-22.86" size="1.778" layer="96"/>
+</instance>
+<instance part="RP1" gate="B" x="40.64" y="-10.16" smashed="yes">
 <attribute name="NAME" x="43.18" y="-10.16" size="1.778" layer="95"/>
 <attribute name="VALUE" x="50.8" y="-10.16" size="1.778" layer="96"/>
 </instance>
-<instance part="RP1" gate="B" x="40.64" y="-7.62" smashed="yes">
+<instance part="RP1" gate="C" x="40.64" y="-7.62" smashed="yes">
 <attribute name="NAME" x="43.18" y="-7.62" size="1.778" layer="95"/>
 <attribute name="VALUE" x="50.8" y="-7.62" size="1.778" layer="96"/>
 </instance>
-<instance part="RP1" gate="C" x="40.64" y="-5.08" smashed="yes">
+<instance part="RP1" gate="D" x="40.64" y="-5.08" smashed="yes">
 <attribute name="NAME" x="43.18" y="-5.08" size="1.778" layer="95"/>
 <attribute name="VALUE" x="50.8" y="-5.08" size="1.778" layer="96"/>
 </instance>
-<instance part="RP1" gate="D" x="63.5" y="-22.86"/>
 <instance part="SUPPLY11" gate="GND" x="-111.76" y="27.94"/>
 <instance part="HD2" gate="A" x="109.22" y="-20.32"/>
@@
 </segment>
 </net>
-<net name="RST" class="0">
-<segment>
-<pinref part="U1" gate="P" pin="PC6(RESET)"/>
-<wire x1="-33.02" y1="25.4" x2="-38.1" y2="25.4" width="0.1524" layer="91"/>
-<label x="-38.1" y="25.4" size="1.778" layer="95" font="vector" rot="R180"/>
-</segment>
-<segment>
-<wire x1="114.3" y1="-22.86" x2="119.38" y2="-22.86" width="0.1524" layer="91"/>
-<label x="119.38" y="-22.86" size="1.778" layer="95" font="vector"/>
-<pinref part="HD2" gate="A" pin="5"/>
-</segment>
-</net>
 <net name="AREF" class="0">
 <segment>
@@
 <net name="RR-" class="0">
 <segment>
+<pinref part="U1" gate="P" pin="PB0(ICP1)"/>
+<pinref part="RP1" gate="D" pin="2"/>
+</segment>
+</net>
+<net name="RG-" class="0">
+<segment>
+<pinref part="U1" gate="P" pin="PB1(OC1A)"/>
 <pinref part="RP1" gate="C" pin="2"/>
-<pinref part="U1" gate="P" pin="PB0(ICP1)"/>
-</segment>
-</net>
-<net name="RG-" class="0">
-<segment>
+</segment>
+</net>
+<net name="RB-" class="0">
+<segment>
+<pinref part="U1" gate="P" pin="PB2(SS/OC1B)"/>
 <pinref part="RP1" gate="B" pin="2"/>
-<pinref part="U1" gate="P" pin="PB1(OC1A)"/>
-</segment>
-</net>
-<net name="RB-" class="0">
-<segment>
-<pinref part="RP1" gate="A" pin="2"/>
-<pinref part="U1" gate="P" pin="PB2(SS/OC1B)"/>
 </segment>
 </net>
 <net name="R-" class="0">
 <segment>
+<pinref part="D1" gate="A" pin="R-"/>
+<pinref part="RP1" gate="D" pin="1"/>
+<wire x1="45.72" y1="-5.08" x2="55.88" y2="-5.08" width="0.1524" layer="91"/>
+</segment>
+</net>
+<net name="G-" class="0">
+<segment>
+<pinref part="D1" gate="A" pin="G-"/>
 <pinref part="RP1" gate="C" pin="1"/>
-<pinref part="D1" gate="A" pin="R-"/>
-<wire x1="45.72" y1="-5.08" x2="55.88" y2="-5.08" width="0.1524" layer="91"/>
-</segment>
-</net>
-<net name="G-" class="0">
-<segment>
+<wire x1="45.72" y1="-7.62" x2="55.88" y2="-7.62" width="0.1524" layer="91"/>
+</segment>
+</net>
+<net name="B-" class="0">
+<segment>
+<pinref part="D1" gate="A" pin="B-"/>
 <pinref part="RP1" gate="B" pin="1"/>
-<pinref part="D1" gate="A" pin="G-"/>
-<wire x1="45.72" y1="-7.62" x2="55.88" y2="-7.62" width="0.1524" layer="91"/>
-</segment>
-</net>
-<net name="B-" class="0">
-<segment>
-<pinref part="RP1" gate="A" pin="1"/>
-<pinref part="D1" gate="A" pin="B-"/>
 <wire x1="45.72" y1="-10.16" x2="55.88" y2="-10.16" width="0.1524" layer="91"/>
 </segment>
@@
 </sheet>
 </sheets>
-<errors>
-</errors>
 </schematic>
 </drawing>
